Commit message: fixing problem moving right finger

File: urdf/robotiq_hand_e_macro.urdf.xacro (robot description, xacro)
@@ -119,5 +119,5 @@
         <child link="${prefix}hande_right_finger"/>
         <axis xyz="1 0 0"/>
-        <limit effort="200.0" lower="0.0" upper="${gripper_maximal_stroke/2}" velocity="0.15"/>
+        <limit effort="200.0" lower="-10000.0" upper="${gripper_maximal_stroke/2}" velocity="0.15"/>
         <dynamics damping="1.0" friction="0.1"/>
       </joint>
